File: pcb.sch (EAGLE design)
At the start: 22 parts, among them J3 POWER_JACKPTH_BREAD, U1 BOB-12009

Commit message: Modified design so that it respects the height constraint
Parts:
- removed JP3: (no value), pinhead:PINHD-1X2
- removed U1: BOB-12009, BOB-12009:BOB-12009
- added CONN_1: (no value), pinhead:PINHD-2X17
- added JP4: (no value), pinhead:PINHD-1X6/90
- JP1: device pinhead:PINHD-2X17 -> pinhead:PINHD-1X2
Connections:
- removed net 3.3V: JP2.4, U1.LV
- removed net D4: J2.7, J52.7, U$10.Z
- removed net D5: J2.8, J52.8, U$10.S0
- removed net D6: J2.9, J52.9, U$10.S1
- removed net D7: J2.10, J52.10, U$10.S2
- removed net D8: 1.SCK, 2.SCK, 3.SCK, 4.SCK, 5.SCK, 6.SCK, 7.SCK, 8.SCK, J2.11, J52.11
- removed net RX: JP2.2, U1.LV2
- removed net TX: JP2.3, U1.LV1
- new net D4/Z: J2.7, J52.7, JP4.5, U$10.Z
- new net D5/S0: J2.8, J52.8, JP4.4, U$10.S0
- new net D6/S1: J2.9, J52.9, JP4.3, U$10.S1
- new net D7/S2: J2.10, J52.10, JP4.2, U$10.S2
- new net D8/HX711_SCK: 1.SCK, 2.SCK, 3.SCK, 4.SCK, 5.SCK, 6.SCK, 7.SCK, 8.SCK, J2.11, J52.11, JP4.6
- net 5.0V: now also JP2.4; no longer U1.HV
- net A+1: now also CONN_1.3; no longer JP1.3
- net A+2: now also CONN_1.7; no longer JP1.7
- net A+3: now also CONN_1.11; no longer JP1.11
- net A+4: now also CONN_1.15; no longer JP1.15
- net A+5: now also CONN_1.19; no longer JP1.19
- net A+6: now also CONN_1.23; no longer JP1.23
- net A+7: now also CONN_1.27; no longer JP1.27
- net A+8: now also CONN_1.31; no longer JP1.31
- net A-1: now also CONN_1.4; no longer JP1.4
- net A-2: now also CONN_1.8; no longer JP1.8
- net A-3: now also CONN_1.12; no longer JP1.12
- net A-4: now also CONN_1.16; no longer JP1.16
- net A-5: now also CONN_1.20; no longer JP1.20
- net A-6: now also CONN_1.24; no longer JP1.24
- net A-7: now also CONN_1.28; no longer JP1.28
- net A-8: now also CONN_1.32; no longer JP1.32
- net D2: no longer U1.HV2
- net D3: no longer U1.HV1
- net E+1: now also CONN_1.1; no longer JP1.1
- net E+2: now also CONN_1.5; no longer JP1.5
- net E+3: now also CONN_1.9; no longer JP1.9
- net E+4: now also CONN_1.13; no longer JP1.13
- net E+5: now also CONN_1.17; no longer JP1.17
- net E+6: now also CONN_1.21; no longer JP1.21
- net E+7: now also CONN_1.25; no longer JP1.25
- net E+8: now also CONN_1.29; no longer JP1.29
- net E-1: now also CONN_1.2; no longer JP1.2
- net E-2: now also CONN_1.6; no longer JP1.6
- net E-3: now also CONN_1.10; no longer JP1.10
- net E-4: now also CONN_1.14; no longer JP1.14
- net E-5: now also CONN_1.18; no longer JP1.18
- net E-6: now also CONN_1.22; no longer JP1.22
- net E-7: now also CONN_1.26; no longer JP1.26
- net E-8: now also CONN_1.30; no longer JP1.30
- net GND: now also JP4.1; no longer U1.GND
- net P1: now also CONN_1.34, JP1.1; no longer JP1.34, JP3.1
- net P2: now also CONN_1.33, JP1.2; no longer JP1.33, JP3.2
- net RX0: now also JP2.2
- net TX1: now also JP2.3
Other:
- note removed: "LLC"
- moved on the sheet: 1, 2, 3, 5, 6, 7, D2, D3, J3, JP2, R1, R2
